File: Xiegu MiniMic.kicad_pcb (KiCad board)
At the start: 2 copper layers, 50.8 x 25.4 mm, 22 parts, among them J1 54602-908LF

Commit message: Rev B
Parts:
- turned MK1 to 180 degrees
Connections:
- MK1 pad 1: MIC-GND -> Net-(C1-Pad1)
- MK1 pad 2: Net-(C1-Pad1) -> MIC-GND
Routing:
- net MIC-GND: track 36.9 -> 32.6 mm
- net Net-(C1-Pad1): track 18.4 -> 15.9 mm
Other:
- board text added: "Rev. B"
- board text removed: "Rev. A"
Changed lines of the file:
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@@
       (drillshape 0)
       (scaleselection 1)
-      (outputdirectory "ASSEMBLY/")
+      (outputdirectory "GERBER/")
     )
   )
@@
     (tags "inductor")
     (property "Digikey PN" "445-16476-1-ND")
-    (property "LCSC PN" "C295130")
+    (property "LCSC" "C295130")
+    (property "LCSC PN" "")
     (property "MPN" "NLV25T-330J-EF")
     (property "Manufacturer" "TDK Corporation")
@@
     (tags "capacitor")
     (property "Digikey PN" "478-1308-1-ND")
-    (property "LCSC PN" "C1804")
+    (property "LCSC" "C1804")
+    (property "LCSC PN" "")
     (property "MPN" "08055A220JAT2A")
     (property "Manufacturer" "KYOCERA AVX")
@@
     (tags "resistor")
     (property "Digikey PN" "A106060CT-ND")
-    (property "LCSC PN" "C2073912")
+    (property "LCSC" "C2073912")
+    (property "LCSC PN" "")
     (property "MPN" "CRG0805F2K2")
     (property "Manufacturer" "TE Connectivity Passive Product")
@@
     (tags "capacitor")
     (property "Digikey PN" "478-5034-1-ND")
-    (property "LCSC PN" "C28323")
+    (property "LCSC" "C28323")
+    (property "LCSC PN" "")
     (property "MPN" "0805YC105KAT2A")
     (property "Manufacturer" "KYOCERA AVX")
@@
     (tags "capacitor")
     (property "Digikey PN" "478-1308-1-ND")
-    (property "LCSC PN" "C1804")
+    (property "LCSC" "C1804")
+    (property "LCSC PN" "")
     (property "MPN" "08055A220JAT2A")
     (property "Manufacturer" "KYOCERA AVX")
@@
     (tags "capacitor")
     (property "Digikey PN" "478-1324-1-ND")
-    (property "LCSC PN" "C1743")
+    (property "LCSC" "C1743")
+    (property "LCSC PN" "")
     (property "MPN" "08055A471JAT2A")
     (property "Manufacturer" "KYOCERA AVX")
@@
     (tags "capacitor")
     (property "Digikey PN" "478-08055C472K4T4ACT-ND")
-    (property "LCSC PN" "C1744")
+    (property "LCSC" "C1744")
+    (property "LCSC PN" "")
     (property "MPN" "08055C472K4T4A")
     (property "Manufacturer" "KYOCERA AVX")
@@
     (tags "capacitor")
     (property "Digikey PN" "478-10836-1-ND")
-    (property "LCSC PN" "C28233")
+    (property "LCSC" "C28233")
+    (property "LCSC PN" "")
     (property "MPN" "08055C104KAT4A")
     (property "Manufacturer" "KYOCERA AVX")
@@
     (at 109.22 85.7605)
     (property "Digikey PN" "450-1658-ND")
-    (property "LCSC PN" "C266183")
+    (property "LCSC" "C266183")
+    (property "LCSC PN" "")
     (property "MPN" "1-1825027-1")
     (property "Manufacturer" "TE Connectivity ALCOSWITCH Switches")
@@
     (tags "capacitor")
     (property "Digikey PN" "478-10836-1-ND")
-    (property "LCSC PN" "C28233")
+    (property "LCSC" "C28233")
+    (property "LCSC PN" "")
     (property "MPN" "08055C104KAT4A")
     (property "Manufacturer" "KYOCERA AVX")
@@
     (tags "capacitor")
     (property "Digikey PN" "478-08055C472K4T4ACT-ND")
-    (property "LCSC PN" "C1744")
+    (property "LCSC" "C1744")
+    (property "LCSC PN" "")
     (property "MPN" "08055C472K4T4A")
     (property "Manufacturer" "KYOCERA AVX")
@@
     (tags "RJ45")
     (property "Digikey PN" "609-1046-ND")
-    (property "LCSC PN" "N/A")
+    (property "LCSC" "N/A")
+    (property "LCSC PN" "")
     (property "MPN" "54602-908LF")
     (property "Manufacturer" "Amphenol ICC (FCI)")
@@
     (tags "SOD-123")
     (property "Digikey PN" "MMSZ5239B-FDICT-ND")
-    (property "LCSC PN" "C459546")
+    (property "LCSC" "C459546")
+    (property "LCSC PN" "")
     (property "MPN" "MMSZ5239B-7-F")
     (property "Manufacturer" "Diodes Incorporated")
@@
     (tags "capacitor")
     (property "Digikey PN" "478-1308-1-ND")
-    (property "LCSC PN" "C1804")
+    (property "LCSC" "C1804")
+    (property "LCSC PN" "")
     (property "MPN" "08055A220JAT2A")
     (property "Manufacturer" "KYOCERA AVX")
@@
     (tags "resistor")
     (property "Digikey PN" "A106060CT-ND")
-    (property "LCSC PN" "C2073912")
+    (property "LCSC" "C2073912")
+    (property "LCSC PN" "")
     (property "MPN" "CRG0805F2K2")
     (property "Manufacturer" "TE Connectivity Passive Product")
@@
     (tags "SOD-123")
     (property "Digikey PN" "MMSZ5239B-FDICT-ND")
-    (property "LCSC PN" "C459546")
+    (property "LCSC" "C459546")
+    (property "LCSC PN" "")
     (property "MPN" "MMSZ5239B-7-F")
     (property "Manufacturer" "Diodes Incorporated")
@@
     (tags "capacitor electrolytic")
     (property "Digikey PN" "493-2173-1-ND")
-    (property "LCSC PN" "C445074")
+    (property "LCSC" "C445074")
+    (property "LCSC PN" "")
     (property "MPN" "UWT1C100MCL1GB")
     (property "Manufacturer" "Nichicon")
@@
   )
   (footprint "Xiegu MiniMic:EM6022P" (layer "B.Cu")
-    (at 104.14 76.3625)
+    (at 104.14 76.3625 180)
     (property "Digikey PN" "433-1088-ND")
-    (property "LCSC PN" "N/A")
+    (property "LCSC" "N/A")
+    (property "LCSC PN" "")
     (property "MPN" "EM-6022P")
     (property "Manufacturer" "Soberton Inc.")
@@
     (property "Sheetname" "")
     (attr through_hole)
-    (fp_text reference "MK1" (at -1.287 -0.127 -90 unlocked) (layer "B.SilkS")
+    (fp_text reference "MK1" (at -1.287 -0.127 90 unlocked) (layer "B.SilkS")
       (effects (font (size 1 1) (thickness 0.15)) (justify mirror))
     )
-    (fp_text value "EM6022P" (at 0 -4 180 unlocked) (layer "B.Fab")
+    (fp_text value "EM6022P" (at 0 -4 unlocked) (layer "B.Fab")
       (effects (font (size 1 1) (thickness 0.15)) (justify mirror))
     )
-    (fp_text user "${REFERENCE}" (at 0 4 180 unlocked) (layer "B.Fab")
+    (fp_text user "${REFERENCE}" (at 0 4 unlocked) (layer "B.Fab")
       (effects (font (size 1 1) (thickness 0.15)) (justify mirror))
     )
     (fp_circle (center 0 0) (end 3 0) (layer "B.SilkS") (width 0.12) (fill none))
-    (pad "1" thru_hole circle (at 0.9 -0.95) (size 1.3 1.3) (drill 0.65) (layers *.Cu *.Mask)
-      (net 2 "MIC-GND") (pinfunction "-") (pintype "passive"))
-    (pad "2" thru_hole circle (at 0.9 0.95) (size 1.3 1.3) (drill 0.65) (layers *.Cu *.Mask)
-      (net 1 "Net-(C1-Pad1)") (pinfunction "+") (pintype "passive"))
+    (pad "1" thru_hole circle (at 0.9 -0.95 180) (size 1.3 1.3) (drill 0.65) (layers *.Cu *.Mask)
+      (net 1 "Net-(C1-Pad1)") (pinfunction "-") (pintype "passive"))
+    (pad "2" thru_hole circle (at 0.9 0.95 180) (size 1.3 1.3) (drill 0.65) (layers *.Cu *.Mask)
+      (net 2 "MIC-GND") (pinfunction "+") (pintype "passive"))
     (model "${KIPRJMOD}/Xiegu MiniMic.pretty/EM-6022P-1.step"
       (offset (xyz 0 0 0))
@@
   )
   (gr_rect (start 68.58 63.6625) (end 119.38 89.0625) (layer "Edge.Cuts") (width 0.1) (fill none))
-  (gr_text "Rev. A" (at 78.74 66.2025) (layer "F.SilkS")
+  (gr_text "Rev. B" (at 78.74 66.2025) (layer "F.SilkS")
     (effects (font (size 1 1) (thickness 0.15)))
   )
@@
     (style (thickness 0.15) (arrow_length 1.27) (text_position_mode 0) (extension_height 0.58642) (extension_offset 0.5) keep_text_aligned)
   )
-  (segment (start 105.04 77.3125) (end 105.04 78.8466) (width 0.635) (layer "F.Cu") (net 1))
   (segment (start 98.298 80.8075) (end 98.298 78.7265) (width 0.635) (layer "F.Cu") (net 1))
-  (segment (start 105.04 78.8466) (end 103.14 80.7466) (width 0.635) (layer "F.Cu") (net 1))
+  (segment (start 103.24 77.3125) (end 103.24 80.6466) (width 0.635) (layer "F.Cu") (net 1))
   (segment (start 96.647 81.5321) (end 97.5734 81.5321) (width 0.635) (layer "F.Cu") (net 1))
-  (segment (start 99.712 77.3125) (end 105.04 77.3125) (width 0.635) (layer "F.Cu") (net 1))
+  (segment (start 99.712 77.3125) (end 103.24 77.3125) (width 0.635) (layer "F.Cu") (net 1))
+  (segment (start 103.24 80.6466) (end 103.14 80.7466) (width 0.635) (layer "F.Cu") (net 1))
   (segment (start 95.0805 81.5321) (end 94.168 80.6196) (width 0.635) (layer "F.Cu") (net 1))
   (segment (start 98.298 78.7265) (end 99.712 77.3125) (width 0.635) (layer "F.Cu") (net 1))
@@
   (segment (start 90.866 76.1746) (end 89.916 75.2246) (width 0.635) (layer "F.Cu") (net 2))
   (segment (start 94.615 77.6325) (end 94.2729 77.6325) (width 0.635) (layer "F.Cu") (net 2))
-  (segment (start 99.712 75.4125) (end 105.04 75.4125) (width 0.635) (layer "F.Cu") (net 2))
-  (segment (start 105.04 72.9445) (end 103.124 71.0285) (width 0.635) (layer "F.Cu") (net 2))
   (segment (start 92.815 76.1746) (end 90.866 76.1746) (width 0.635) (layer "F.Cu") (net 2))
   (segment (start 94.2729 77.6325) (end 92.815 76.1746) (width 0.635) (layer "F.Cu") (net 2))
   (segment (start 85.4761 76.9975) (end 87.249 75.2246) (width 0.635) (layer "F.Cu") (net 2))
-  (segment (start 105.04 75.4125) (end 105.04 72.9445) (width 0.635) (layer "F.Cu") (net 2))
   (segment (start 87.249 75.2246) (end 89.916 75.2246) (width 0.635) (layer "F.Cu") (net 2))
+  (segment (start 103.24 71.1445) (end 103.124 71.0285) (width 0.635) (layer "F.Cu") (net 2))
+  (segment (start 103.24 75.4125) (end 103.24 71.1445) (width 0.635) (layer "F.Cu") (net 2))
+  (segment (start 103.24 75.4125) (end 99.712 75.4125) (width 0.635) (layer "F.Cu") (net 2))
   (segment (start 81.3 76.9975) (end 85.4761 76.9975) (width 0.635) (layer "F.Cu") (net 2))
   (via (at 94.615 77.6325) (size 0.8) (drill 0.4) (layers "F.Cu" "B.Cu") (net 2))
-  (segment (start 105.04 75.4125) (end 102.82 77.6325) (width 0.635) (layer "B.Cu") (net 2))
-  (segment (start 102.82 77.6325) (end 102.235 77.6325) (width 0.635) (layer "B.Cu") (net 2))
-  (segment (start 102.235 77.6325) (end 94.615 77.6325) (width 0.635) (layer "B.Cu") (net 2))
+  (segment (start 101.274 77.3785) (end 94.869 77.3785) (width 0.635) (layer "B.Cu") (net 2))
+  (segment (start 94.869 77.3785) (end 94.615 77.6325) (width 0.635) (layer "B.Cu") (net 2))
+  (segment (start 103.24 75.4125) (end 101.274 77.3785) (width 0.635) (layer "B.Cu") (net 2))
   (segment (start 87.2439 79.6645) (end 87.249 79.6696) (width 0.635) (layer "F.Cu") (net 3))
   (segment (start 83.84 78.2675) (end 85.237 79.6645) (width 0.635) (layer "F.Cu") (net 3))
