File: Xiegu MiniMic.kicad_sch (KiCad schematic)
At the start: 22 parts, among them J1 54602-908LF

Commit message: Rev B
Connections:
- net MIC-GND: now also MK1.2 (+); no longer MK1.1 (-)
- net at C1.1, C2.1, D2.1 (K)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: now also MK1.1 (-); no longer MK1.2 (+)
Other:
- moved on the sheet: MK1
Changed lines of the file:
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@@
   (title_block
     (title "Xiegu Mini Hand Mic")
-    (date "2022-11-08")
-    (rev "A")
+    (date "2022-11-15")
+    (rev "B")
     (company "Jonathan Kayne, KM4CFT")
     (comment 1 "Based on the ICOM HM151")
@@
     (pin "1")
   )
-  (symbol (lib_id "Device:Microphone_Condenser") (at 88.9 88.9 0) (unit 1)
-    (in_bom yes) (on_board yes)
-    (property "Reference" "MK1" (id 0) (at 85.598 87.63 0)
+  (symbol (lib_id "Device:Microphone_Condenser") (at 88.9 88.9 180) (unit 1)
+    (in_bom yes) (on_board yes)
+    (property "Reference" "MK1" (id 0) (at 81.28 90.17 0)
       (effects (font (size 1.27 1.27)) (justify right))
     )
-    (property "Value" "EM6022P" (id 1) (at 85.598 89.535 0)
+    (property "Value" "EM6022P" (id 1) (at 77.47 87.63 0)
       (effects (font (size 1.27 1.27)) (justify right))
     )
-    (property "Footprint" "Xiegu MiniMic:EM6022P" (id 2) (at 88.9 86.36 90)
-      (effects (font (size 1.27 1.27)) hide)
-    )
-    (property "Datasheet" "~" (id 3) (at 88.9 86.36 90)
-      (effects (font (size 1.27 1.27)) hide)
-    )
+    (property "Footprint" "Xiegu MiniMic:EM6022P" (id 2) (at 88.9 91.44 90)
+      (effects (font (size 1.27 1.27)) hide)
+    )
+    (property "Datasheet" "~" (id 3) (at 88.9 91.44 90)
+      (effects (font (size 1.27 1.27)) hide)
+    )
